File: Hardware/ADS1299.sch (KiCad schematic (older format))
At the start: 32 parts, among them J2 IOs Multipropósito, U10 ADS1299, U14 OPA2376

Commit message: Listado de materiales con precios DIGIKEY 01/2018
Parts:
- U14: Footprint 8-SOIC (0.154\", 3.90mm Width) -> 8-SOIC (0.154\" 3.90mm Width)
Changed lines of the file:
@@
 F 6 "OPA2376AIDR" H 2800 1700 60  0001 C CNN "Nro de parte"
 F 7 "296-22564-1-ND" H 2800 1700 60  0001 C CNN "Digikey"
-F 8 "8-SOIC (0.154\", 3.90mm Width)" H 2800 1700 60  0001 C CNN "Footprint"
+F 8 "8-SOIC (0.154\" 3.90mm Width)" H 2800 1700 60  0001 C CNN "Footprint"
 	1    2900 1300
 	-1   0    0    -1
@@
 F 6 "OPA2376AIDR" H 2800 1700 60  0001 C CNN "Nro de parte"
 F 7 "296-22564-1-ND" H 2800 1700 60  0001 C CNN "Digikey"
-F 8 "8-SOIC (0.154\", 3.90mm Width)" H 2800 1700 60  0001 C CNN "Footprint"
+F 8 "8-SOIC (0.154\" 3.90mm Width)" H 2800 1700 60  0001 C CNN "Footprint"
 	2    1550 2950
 	1    0    0    -1
