File: Hardware/Aislación.sch (KiCad schematic (older format))
At the start: 36 parts, among them U11 ADuM6401, U12 ADuM2401, U13 NCP1117ST33T3G

Commit message: Listado de materiales con precios DIGIKEY 01/2018
Parts:
- U11, U12: Footprint 16-SOIC (0.295\", 7.50mm Width) -> 16-SOIC (0.295\" 7.50mm Width)
Changed lines of the file:
@@
 F 6 "ADUM6401CRWZ" H 2800 1700 60  0001 C CNN "Nro de parte"
 F 7 "ADUM6401CRWZ-ND" H 2800 1700 60  0001 C CNN "Digikey"
-F 8 "16-SOIC (0.295\", 7.50mm Width)	" H 2800 1700 60  0001 C CNN "Footprint"
+F 8 "16-SOIC (0.295\" 7.50mm Width)	" H 2800 1700 60  0001 C CNN "Footprint"
 	1    5100 1950
 	-1   0    0    -1
@@
 F 6 "ADUM2401ARWZ-RL" H 2800 1700 60  0001 C CNN "Nro de parte"
 F 7 "ADUM2401ARWZ-RLCT-ND" H 2800 1700 60  0001 C CNN "Digikey"
-F 8 "16-SOIC (0.295\", 7.50mm Width)" H 2800 1700 60  0001 C CNN "Footprint"
+F 8 "16-SOIC (0.295\" 7.50mm Width)" H 2800 1700 60  0001 C CNN "Footprint"
 	1    5125 3400
 	-1   0    0    -1
