File: Hardware/Protección.sch (KiCad schematic (older format))
At the start: 51 parts, among them J1 20POS SIL VERTICAL PIN HEADER, U1 TPD2E001, U15 TPD2E001, U2 TPD2E001, U3 TPD2E001, U4 TPD2E001, U5 TPD2E001, U6 TPD2E001, U7 TPD2E001, U8 TPD2E001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

Commit message: Listado de materiales con precios DIGIKEY 01/2018
Parts:
- J1: Descripción 20 Positions Header, Cuttable Connector 0.100\" (2.54mm) Th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 -> Cuttable Connector 0.100\" (2.54mm) Through Hole Tin
- R13: Código Digikey 311-2.2KARCT-ND -> (none); Descripción (none) -> RES SMD 2.2K OHM 5% 1/8W 0805
Changed lines of the file:
@@
 F 2 "" H 2950 5300 60  0001 C CNN
 F 3 "PYu-RC_Group_51_RoHS_L_8.pdf" H 2800 1700 60  0001 C CNN
-F 4 "311-2.2KARCT-ND" V 2950 5300 60  0001 C CNN "Código Digikey"
+F 4 "RES SMD 2.2K OHM 5% 1/8W 0805" V 2950 5300 60  0001 C CNN "Descripción"
 F 5 "Yageo" H 2800 1700 60  0001 C CNN "Fabricante"
 F 6 "RC0805JR-072K2L" H 2800 1700 60  0001 C CNN "Nro de parte"
@@
 F 2 "footprints:Pin_Header_Straight_1x20" H 1300 1750 60  0001 C CNN
 F 3 "M20-999.pdf" H 1300 1750 60  0001 C CNN
-F 4 "20 Positions Header, Cuttable Connector 0.100\" (2.54mm) Through Hole Tin" H 1300 1750 60  0001 C CNN "Descripción"
+F 4 "Cuttable Connector 0.100\" (2.54mm) Through Hole Tin" H 1300 1750 60  0001 C CNN "Descripción"
 F 5 "Harwin Inc." H 1300 1750 60  0001 C CNN "Fabricante"
 F 6 "M20-9992046" H 1300 1750 60  0001 C CNN "Nro de parte"
