File: Hardware/PonchoBiopotenciales.kicad_pcb (KiCad board)
At the start: 2 copper layers, 85.9 x 80.5 mm, 120 parts, among them J1 Entradas Analógicas, J2 IOs Multipropósito, U1 TPD2E001, U10 ADS1299, U11 ADuM6401, U12 ADuM2401, U13 NCP1117ST33T3G, U14 OPA2376, U15 TPD2E001, U2 TPD2E001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

Commit message: corregidos los slots de los ADUM
Parts:
- removed SC_1: Slot_1, footprints:Fiducial_1mm_Dia_2.54mm_Outer_CopperTop
- removed SC_2: Slot_2, footprints:Fiducial_1mm_Dia_2.54mm_Outer_CopperTop
Other:
- outline, holes or cut-outs redrawn
